File: intellivision/project/intellivision-mod.kicad_pcb (KiCad board)
At the start: 2 copper layers, 32.5 x 33.5 mm, 0 parts

Commit message: Cleaner version
Routing:
- net (no net): track 0.00 -> 200.7 mm
- net 0: track 200.7 -> 0.00 mm
