File: intellivision/project/kicad/intellivision-composite-rebuilt.kicad_sch (KiCad schematic)
At the start: 21 parts, among them J1 VID IN, J2 VID OUT, J3 AUD IN, J4 AUD OUT, J5 +5V IN, J6 GND IN, J7 GND OUT, Q1 2N3904, Q2 2N3904

Commit message: Add routing
Connections:
- net GND: now also J6.1 (Pin_1), J7.1 (Pin_1), R4.2, R6.2, R8.2
- net at J1.1 (Pin_1): now also C1.1; no longer C1.2
- net at Q1.2 (B): now also C1.2; no longer C1.1
Other:
- moved on the sheet: C1
Changed lines of the file:
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@@
+	)
+	(junction
+		(at 102.87 101.6)
+		(diameter 0)
+		(color 0 0 0 0)
 	)
 	(junction
@@
 	(wire
 		(pts
+			(xy 102.87 101.6) (xy 193.04 101.6)
+		)
+		(stroke
+			(width 0)
+			(type default)
+		)
+	)
+	(wire
+		(pts
 			(xy 181.61 71.12) (xy 193.04 71.12)
 		)
@@
 	(wire
 		(pts
-			(xy 76.2 101.6) (xy 193.04 101.6)
+			(xy 76.2 101.6) (xy 102.87 101.6)
 		)
 		(stroke
@@
 	(symbol
 		(lib_id "Device:C_Polarized")
-		(at 71.12 76.2 270)
+		(at 71.12 76.2 90)
+		(mirror x)
 		(unit 1)
 		(body_style 1)
@@
 			)
 		)
-			(property "Footprint" "Intellivision:TO-92_Inline_OAR175"
+		(property "Footprint" "Intellivision:TO-92_Inline_OAR175"
 			(at 116.84 76.2 0)
 			(hide yes)
@@
 			)
 		)
-			(property "Footprint" "Intellivision:TO-92_Inline_OAR175"
+		(property "Footprint" "Intellivision:TO-92_Inline_OAR175"
 			(at 157.48 76.2 0)
 			(hide yes)
@@
 					(unit 1)
 				)
+			)
+		)
+	)
+	(symbol
+		(lib_id "power:GND")
+		(at 102.87 101.6 0)
+		(unit 1)
+		(body_style 1)
+		(exclude_from_sim no)
+		(in_bom yes)
+		(on_board yes)
+		(in_pos_files yes)
+		(dnp no)
+		(fields_autoplaced yes)
+		(property "Reference" "#PWR03"
+			(at 102.87 107.95 0)
+			(hide yes)
+			(show_name no)
+			(do_not_autoplace no)
+			(effects
+				(font
+					(size 1.27 1.27)
+				)
+			)
+		)
+		(property "Value" "GND"
+			(at 102.87 106.68 0)
+			(show_name no)
+			(do_not_autoplace no)
+			(effects
+				(font
+					(size 1.27 1.27)
+				)
+			)
+		)
+		(property "Footprint" ""
+			(at 102.87 101.6 0)
+			(hide yes)
+			(show_name no)
+			(do_not_autoplace no)
+			(effects
+				(font
+					(size 1.27 1.27)
+				)
+			)
+		)
+		(property "Datasheet" ""
+			(at 102.87 101.6 0)
+			(hide yes)
+			(show_name no)
+			(do_not_autoplace no)
+			(effects
+				(font
+					(size 1.27 1.27)
+				)
+			)
+		)
+		(property "Description" "Power symbol creates a global label with name \"GND\" , ground"
+			(at 102.87 101.6 0)
+			(hide yes)
+			(show_name no)
+			(do_not_autoplace no)
+			(effects
+				(font
+					(size 1.27 1.27)
+				)
+			)
+		)
+		(pin "1"
+		)
+		(instances
+			(project "intellivision-composite-rebuilt"
+				(path "/47fa711f-e952-4277-8d24-ac8ef3d4e81c"
+					(reference "#PWR03")
+					(unit 1)
+				)
