File: intellivision/project/kicad/intv-video-composite.kicad_pcb (KiCad board)
At the start: 2 copper layers, 35.5 x 33.5 mm, 21 parts, among them J1 VID IN, J2 VID OUT, J3 AUD IN, J4 AUD OUT, J5 +5V IN, J6 GND IN, J7 GND OUT, Q1 2N3904, Q2 2N3904

Commit message: De way i like it
Parts:
- J1: value VID IN -> VIDEO IN
- J2: value VID OUT -> VIDEO OUT
- J3: value AUD IN -> AUDIO IN
- J4: value AUD OUT -> AUDIO OUT
Other:
- board text removed: "+"
